Commit message: pi0 deploy

File: install/workcell_config/share/workcell_config/config/workcell.ros2_control.xacro (robot description, xacro)
@@ -1,5 +1,5 @@
 <?xml version="1.0"?>
 <robot xmlns:xacro="http://www.ros.org/wiki/xacro">
-    <xacro:macro name="workcell_ros2_control" params="name use_fake_hardware:=true rws_ip rws_port configure_via_rws:=true initial_positions_file">
+    <xacro:macro name="workcell_ros2_control" params="name use_fake_hardware:=true rws_ip rws_port rws_username:='Default User' rws_password:='robotics' robot_controller_id:='IRB6700' configure_via_rws:=true egm_port:=6515 initial_positions_file">
         <xacro:property name="initial_positions" value="${xacro.load_yaml(initial_positions_file)['initial_positions']}"/>
         <ros2_control name="${name}" type="system">
@@ -14,10 +14,11 @@
               <xacro:unless value="${use_fake_hardware}">
                 <plugin>abb_hardware_interface/ABBSystemHardware</plugin>
-                <param name="rws_ip">192.168.1.1</param>
-                <param name="rws_port">80</param>
-                <param name="rws_username">Default User</param>
-                <param name="rws_password">robotics</param>
-                <param name="configure_via_rws">true</param>
-                <param name="egm_port">6515</param>
+                <param name="rws_ip">${rws_ip}</param>
+                <param name="rws_port">${rws_port}</param>
+                <param name="rws_username">${rws_username}</param>
+                <param name="rws_password">${rws_password}</param>
+                <param name="robot_controller_id">${robot_controller_id}</param>
+                <param name="configure_via_rws">${configure_via_rws}</param>
+                <param name="egm_port">${egm_port}</param>
               </xacro:unless>
             </hardware>

File: install/workcell_config/share/workcell_config/config/workcell.urdf.xacro (robot description, xacro)
@@ -7,6 +7,14 @@
   <xacro:arg name="rws_port"         default="80"/>
   <xacro:property name="rws_port"         value="$(arg rws_port)"/>
+  <xacro:arg name="rws_username"     default="Default User"/>
+  <xacro:property name="rws_username"     value="$(arg rws_username)"/>
+  <xacro:arg name="rws_password"     default="robotics"/>
+  <xacro:property name="rws_password"     value="$(arg rws_password)"/>
+  <xacro:arg name="robot_controller_id" default="IRB6700"/>
+  <xacro:property name="robot_controller_id" value="$(arg robot_controller_id)"/>
   <xacro:arg name="configure_via_rws" default="true"/>
   <xacro:property name="configure_via_rws" value="$(arg configure_via_rws)"/>
+  <xacro:arg name="egm_port"         default="6515"/>
+  <xacro:property name="egm_port"         value="$(arg egm_port)"/>
   <xacro:arg name="prefix" default=""/>
   <xacro:arg name="mesh_scale_visual" default="1 1 1"/>
@@ -43,5 +51,9 @@
     rws_ip="${rws_ip}"
     rws_port="${rws_port}"
+    rws_username="${rws_username}"
+    rws_password="${rws_password}"
+    robot_controller_id="${robot_controller_id}"
     configure_via_rws="${configure_via_rws}"
+    egm_port="${egm_port}"
     initial_positions_file="$(find workcell_config)/config/initial_positions.yaml"/>
 </robot>

File: install/workcell_description/share/workcell_description/urdf/workcell.urdf.xacro (robot description, xacro)
@@ -7,6 +7,14 @@
   <xacro:arg name="rws_port"         default="80"/>
   <xacro:property name="rws_port"         value="$(arg rws_port)"/>
+  <xacro:arg name="rws_username"     default="Default User"/>
+  <xacro:property name="rws_username"     value="$(arg rws_username)"/>
+  <xacro:arg name="rws_password"     default="robotics"/>
+  <xacro:property name="rws_password"     value="$(arg rws_password)"/>
+  <xacro:arg name="robot_controller_id" default="IRB6700"/>
+  <xacro:property name="robot_controller_id" value="$(arg robot_controller_id)"/>
   <xacro:arg name="configure_via_rws" default="true"/>
   <xacro:property name="configure_via_rws" value="$(arg configure_via_rws)"/>
+  <xacro:arg name="egm_port"         default="6515"/>
+  <xacro:property name="egm_port"         value="$(arg egm_port)"/>
   <xacro:arg name="prefix" default=""/>
   <xacro:arg name="mesh_scale_visual" default="1 1 1"/>
@@ -37,5 +45,9 @@
     rws_ip="${rws_ip}"
     rws_port="${rws_port}"
+    rws_username="${rws_username}"
+    rws_password="${rws_password}"
+    robot_controller_id="${robot_controller_id}"
     configure_via_rws="${configure_via_rws}"
+    egm_port="${egm_port}"
     initial_positions_file="$(find workcell_config)/config/initial_positions.yaml"/>
 </robot>
