Commit message: Document real ABB EGM workflow and add HMI motion control

File: src/workcell_description/urdf/workcell.urdf.xacro (robot description, xacro)
@@ -39,4 +39,10 @@
         <origin xyz="0.63170595 -0.03808443 -0.12658877" rpy="1.4194238211454702 -1.2500567786472647 -1.3301909060020083"/>
     </joint>
+    <link name="fixed_cam_mount"/>
+    <joint name="base_to_fixed_cam_mount" type="fixed">
+        <parent link="base_link"/>
+        <child  link="fixed_cam_mount"/>
+        <origin xyz="0.30 0.10 1.50" rpy="0 0 3.14159"/>
+    </joint>
   <xacro:include filename="$(find workcell_config)/config/workcell.ros2_control.xacro"/>
   <xacro:workcell_ros2_control
